Commit message: update

File: tiago_ws/src/tiago_robot/tiago_description/urdf/arm/arm.ros2_control.xacro (robot description, xacro)
@@ -13,14 +13,11 @@
  -->
 <robot xmlns:xacro="http://ros.org/wiki/xacro">
-  <xacro:macro name="ros2_control_arm" params="name reduction offset" >
+  <xacro:macro name="ros2_control_arm" params="name reduction:=1.0 offset" >
     <joint name="${name}_joint">
       <command_interface name="position" />
       <command_interface name="velocity" />
       <command_interface name="effort" />
-      <state_interface name="position">
-        <param name="initial_value">0.5</param>
-      </state_interface>
-      <state_interface name="velocity">
-      </state_interface>
+      <state_interface name="position" />
+      <state_interface name="velocity" />
       <state_interface name="effort" />
     </joint>

File: tiago_ws/src/tiago_robot/tiago_description/urdf/arm/wrist.ros2_control.xacro (robot description, xacro)
@@ -18,7 +18,5 @@
       <command_interface name="velocity" />
       <command_interface name="effort" />
-      <state_interface name="position">
-        <param name="initial_value">1.1</param>
-      </state_interface>
+      <state_interface name="position" />
       <state_interface name="velocity" />
       <state_interface name="effort" />
@@ -33,7 +31,5 @@
       <command_interface name="velocity" />
       <command_interface name="effort" />
-      <state_interface name="position">
-        <param name="initial_value">-1.0</param>
-      </state_interface>
+      <state_interface name="position" />
       <state_interface name="velocity" />
       <state_interface name="effort" />
@@ -43,7 +39,5 @@
       <command_interface name="velocity" />
       <command_interface name="effort" />
-      <state_interface name="position">
-        <param name="initial_value">0.3</param>
-      </state_interface>
+      <state_interface name="position" />
       <state_interface name="velocity" />
       <state_interface name="effort" />

File: tiago_ws/src/tiago_robot/tiago_description/urdf/arm/wrist.urdf.xacro (robot description, xacro)
@@ -111,5 +111,5 @@
       <child link="${name}_6_link" />
       <origin xyz="0 0 ${reflect * 0.15}" rpy="${0.0 * deg_to_rad} ${-90.0 * deg_to_rad} ${-90.0 * deg_to_rad}" />
-      <axis xyz="0 0 1" />
+      <axis xyz="0 0 -1" />
       <limit lower="${-wrist_6_range * deg_to_rad}" upper="${wrist_6_range * deg_to_rad}" effort="${wrist_2_max_effort}" velocity="${wrist_2_max_vel}" />
       <dynamics friction="${wrist_friction}" damping="${wrist_damping}"/>

Commit message: Arm tiago moveit

File: tiago_ws/src/tiago_robot/tiago_description/urdf/arm/arm.ros2_control.xacro (robot description, xacro)
@@ -13,11 +13,14 @@
  -->
 <robot xmlns:xacro="http://ros.org/wiki/xacro">
-  <xacro:macro name="ros2_control_arm" params="name reduction:=1.0 offset" >
+  <xacro:macro name="ros2_control_arm" params="name reduction offset" >
     <joint name="${name}_joint">
       <command_interface name="position" />
       <command_interface name="velocity" />
       <command_interface name="effort" />
-      <state_interface name="position" />
-      <state_interface name="velocity" />
+      <state_interface name="position">
+        <param name="initial_value">0.5</param>
+      </state_interface>
+      <state_interface name="velocity">
+      </state_interface>
       <state_interface name="effort" />
     </joint>

File: tiago_ws/src/tiago_robot/tiago_description/urdf/arm/wrist.ros2_control.xacro (robot description, xacro)
@@ -18,5 +18,7 @@
       <command_interface name="velocity" />
       <command_interface name="effort" />
-      <state_interface name="position" />
+      <state_interface name="position">
+        <param name="initial_value">1.1</param>
+      </state_interface>
       <state_interface name="velocity" />
       <state_interface name="effort" />
@@ -31,5 +33,7 @@
       <command_interface name="velocity" />
       <command_interface name="effort" />
-      <state_interface name="position" />
+      <state_interface name="position">
+        <param name="initial_value">-1.0</param>
+      </state_interface>
       <state_interface name="velocity" />
       <state_interface name="effort" />
@@ -39,5 +43,7 @@
       <command_interface name="velocity" />
       <command_interface name="effort" />
-      <state_interface name="position" />
+      <state_interface name="position">
+        <param name="initial_value">0.3</param>
+      </state_interface>
       <state_interface name="velocity" />
       <state_interface name="effort" />

File: tiago_ws/src/tiago_robot/tiago_description/urdf/arm/wrist.urdf.xacro (robot description, xacro)
@@ -111,5 +111,5 @@
       <child link="${name}_6_link" />
       <origin xyz="0 0 ${reflect * 0.15}" rpy="${0.0 * deg_to_rad} ${-90.0 * deg_to_rad} ${-90.0 * deg_to_rad}" />
-      <axis xyz="0 0 -1" />
+      <axis xyz="0 0 1" />
       <limit lower="${-wrist_6_range * deg_to_rad}" upper="${wrist_6_range * deg_to_rad}" effort="${wrist_2_max_effort}" velocity="${wrist_2_max_vel}" />
       <dynamics friction="${wrist_friction}" damping="${wrist_damping}"/>
